File: TE0724_Connector.kicad_sch (KiCad schematic)
At the start: 15 parts, among them J1 SS5-80-3.50-L-D-K-TR, J3 Conn_02x05_Odd_Even, Q1 2N7002KQ-7, Q2 2N7002KQ-7, U4 TPS79933QDDCRQ1

Commit message: added solder bridges and updated BOM
Parts:
- C3, C6: External Part Num (none) -> C3011652; External Part Number GCM188R71H104KA57J -> (none); MPN C3011652 -> GCM188R71H104KA57J
- C5, C7: External Part Num (none) -> C85867; External Part Number GCM31MR71H105KA55L -> (none); MPN C85867 -> GCM31MR71H105KA55L
- J1: External Part Num (none) -> C5292077; External Part Number SS5-80-3.50-L-D-K-TR -> (none); MPN C5292077 -> SS5-80-3.50-L-D-K-TR
- Q1, Q2: External Part Num (none) -> C111971; External Part Number 2N7002KQ-7 -> (none); MPN C111971 -> 2N7002KQ-7
- R2, R7: MANUFACTURER (none) -> Vishay; MPN (none) -> MCS0402MD1000BE100
- R5, R6: MANUFACTURER (none) -> Vishay; MPN (none) -> MCS0402MD1003BE100
- U4: MANUFACTURER (none) -> Texas Instruments; MPN (none) -> TPS79933QDDCRQ1
Changed lines of the file:
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@@
 			)
 		)
+		(property "MANUFACTURER" "Texas Instruments"
+			(at 129.54 167.64 0)
+			(hide yes)
+			(show_name no)
+			(do_not_autoplace no)
+			(effects
+				(font
+					(size 1.27 1.27)
+				)
+			)
+		)
+		(property "MPN" "TPS79933QDDCRQ1"
+			(at 129.54 167.64 0)
+			(hide yes)
+			(show_name no)
+			(do_not_autoplace no)
+			(effects
+				(font
+					(size 1.27 1.27)
+				)
+			)
+		)
 		(pin "2"
 		)
@@
 			)
 		)
-		(property "External Part Number" "SS5-80-3.50-L-D-K-TR "
+		(property "MPN" "SS5-80-3.50-L-D-K-TR "
 			(at 97.79 85.09 0)
 			(hide yes)
@@
 			)
 		)
-		(property "MPN" "C5292077"
+		(property "External Part Num" "C5292077"
 			(at 97.79 85.09 0)
 			(hide yes)
@@
 			)
 		)
-		(property "External Part Number" ""
-			(at 96.52 172.72 0)
-			(hide yes)
-			(show_name no)
-			(do_not_autoplace no)
-			(effects
-				(font
-					(size 1.27 1.27)
-				)
-			)
-		)
 		(property "MPN" ""
 			(at 96.52 172.72 0)
@@
 			)
 		)
-		(property "External Part Number" ""
-			(at 96.52 170.18 0)
-			(hide yes)
-			(show_name no)
-			(do_not_autoplace no)
-			(effects
-				(font
-					(size 1.27 1.27)
-				)
-			)
-		)
 		(property "MPN" ""
 			(at 96.52 170.18 0)
@@
 			)
 		)
-		(property "External Part Number" "GCM188R71H104KA57J"
+		(property "MPN" "GCM188R71H104KA57J"
 			(at 256.54 69.85 0)
 			(hide yes)
@@
 			)
 		)
-		(property "MPN" "C3011652"
+		(property "External Part Num" "C3011652"
 			(at 256.54 69.85 0)
 			(hide yes)
@@
 			)
 		)
+		(property "MANUFACTURER" "Vishay"
+			(at 254 144.78 90)
+			(hide yes)
+			(show_name no)
+			(do_not_autoplace no)
+			(effects
+				(font
+					(size 1.27 1.27)
+				)
+			)
+		)
+		(property "MPN" "MCS0402MD1000BE100"
+			(at 254 144.78 90)
+			(hide yes)
+			(show_name no)
+			(do_not_autoplace no)
+			(effects
+				(font
+					(size 1.27 1.27)
+				)
+			)
+		)
 		(pin "2"
 		)
@@
 			)
 		)
-		(property "External Part Number" "GCM31MR71H105KA55L"
+		(property "MANUFACTURER" "Murata Electronics"
 			(at 163.83 170.18 0)
 			(hide yes)
@@
 			)
 		)
-		(property "MANUFACTURER" "Murata Electronics"
+		(property "MPN" "GCM31MR71H105KA55L"
 			(at 163.83 170.18 0)
 			(hide yes)
@@
 			)
 		)
-		(property "MPN" "C85867"
+		(property "External Part Num" "C85867"
 			(at 163.83 170.18 0)
 			(hide yes)
@@
 			)
 		)
-		(property "External Part Number" "2N7002KQ-7"
+		(property "MANUFACTURER" "DIODES"
 			(at 265.43 144.78 0)
 			(hide yes)
@@
 			)
 		)
-		(property "MANUFACTURER" "DIODES"
+		(property "MPN" "2N7002KQ-7"
 			(at 265.43 144.78 0)
 			(hide yes)
@@
 			)
 		)
-		(property "MPN" "C111971"
+		(property "External Part Num" "C111971"
 			(at 265.43 144.78 0)
 			(hide yes)
@@
 			)
 		)
+		(property "MANUFACTURER" "Vishay"
+			(at 215.9 149.86 0)
+			(hide yes)
+			(show_name no)
+			(do_not_autoplace no)
+			(effects
+				(font
+					(size 1.27 1.27)
+				)
+			)
+		)
+		(property "MPN" "MCS0402MD1003BE100"
+			(at 215.9 149.86 0)
+			(hide yes)
+			(show_name no)
+			(do_not_autoplace no)
+			(effects
+				(font
+					(size 1.27 1.27)
+				)
+			)
+		)
 		(pin "2"
 		)
@@
 			)
 		)
-		(property "External Part Number" "GCM188R71H104KA57J"
+		(property "MANUFACTURER" "Murata Electronics"
 			(at 128.27 176.53 0)
 			(hide yes)
@@
 			)
 		)
-		(property "MANUFACTURER" "Murata Electronics"
+		(property "MPN" "GCM188R71H104KA57J"
 			(at 128.27 176.53 0)
 			(hide yes)
@@
 			)
 		)
-		(property "MPN" "C3011652"
+		(property "External Part Num" "C3011652"
 			(at 128.27 176.53 0)
 			(hide yes)
@@
 			)
 		)
+		(property "MANUFACTURER" "Vishay"
+			(at 209.55 144.78 90)
+			(hide yes)
+			(show_name no)
+			(do_not_autoplace no)
+			(effects
+				(font
+					(size 1.27 1.27)
+				)
+			)
+		)
+		(property "MPN" "MCS0402MD1000BE100"
+			(at 209.55 144.78 90)
+			(hide yes)
+			(show_name no)
+			(do_not_autoplace no)
+			(effects
+				(font
+					(size 1.27 1.27)
+				)
+			)
+		)
 		(pin "2"
 		)
@@
 			)
 		)
-		(property "External Part Number" "2N7002KQ-7"
+		(property "MANUFACTURER" "DIODES"
 			(at 223.52 144.78 0)
 			(hide yes)
@@
 			)
 		)
-		(property "MANUFACTURER" "DIODES"
+		(property "MPN" "2N7002KQ-7"
 			(at 223.52 144.78 0)
 			(hide yes)
@@
 			)
 		)
-		(property "MPN" "C111971"
+		(property "External Part Num" "C111971"
 			(at 223.52 144.78 0)
 			(hide yes)
@@
 			)
 		)
-		(property "External Part Number" "GCM31MR71H105KA55L"
+		(property "MANUFACTURER" "Murata Electronics"
 			(at 119.38 176.53 0)
 			(hide yes)
@@
 			)
 		)
-		(property "MANUFACTURER" "Murata Electronics"
+		(property "MPN" "GCM31MR71H105KA55L"
 			(at 119.38 176.53 0)
 			(hide yes)
@@
 			)
 		)
-		(property "MPN" "C85867"
+		(property "External Part Num" "C85867"
 			(at 119.38 176.53 0)
 			(hide yes)
@@
 			)
 		)
-		(property "External Part Number" ""
-			(at 46.99 167.64 0)
-			(hide yes)
-			(show_name no)
-			(do_not_autoplace no)
-			(effects
-				(font
-					(size 1.27 1.27)
-				)
-			)
-		)
 		(property "MPN" ""
 			(at 46.99 167.64 0)
@@
 			(at 259.08 149.86 0)
 			(hide yes)
+			(show_name no)
+			(do_not_autoplace no)
+			(effects
+				(font
+					(size 1.27 1.27)
+				)
+			)
+		)
+		(property "MANUFACTURER" "Vishay"
+			(at 259.08 149.86 0)
+			(hide yes)
+			(show_name no)
+			(do_not_autoplace no)
+			(effects
+				(font
+					(size 1.27 1.27)
+				)
+			)
+		)
+		(property "MPN" "MCS0402MD1003BE100"
+			(at 259.08 149.86 0)
+			(hide yes)
