File: PC104_Connector.kicad_sch (KiCad schematic)
At the start: 8 parts

Commit message: Reversed RX and TX pins to accommodate altered UART standard
Connections:
- net UART-RXD LS: now also JP3.1 (A); no longer JP4.2 (B)
- net UART-TXD LS: now also JP4.2 (B); no longer JP3.1 (A)
Changed lines of the file:
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@@
 	(wire
 		(pts
-			(xy 137.16 125.73) (xy 137.16 124.46)
+			(xy 137.16 128.27) (xy 137.16 124.46)
 		)
 		(stroke
@@
 		)
 	)
-	(hierarchical_label "UART-RXD LS"
-		(shape output)
+	(hierarchical_label "UART-TXD LS"
+		(shape input)
 		(at 137.16 88.9 90)
 		(effects
@@
 		)
 	)
-	(hierarchical_label "UART-TXD LS"
-		(shape input)
-		(at 137.16 125.73 270)
-		(effects
-			(font
-				(size 1.27 1.27)
-			)
-			(justify right)
-		)
-	)
 	(hierarchical_label "I2C_SCL_CSKB"
 		(shape output)
@@
 		)
 	)
+	(hierarchical_label "UART-RXD LS"
+		(shape output)
+		(at 137.16 128.27 270)
+		(effects
+			(font
+				(size 1.27 1.27)
+			)
+			(justify right)
+		)
+	)
